Commit message: ForReference

File: hros5_description/urdf/modules/arms.xacro (robot description, xacro)
@@ -6,5 +6,5 @@
 			<child link="${side}Shoulder"/>
 			<origin xyz="0.003 ${reflect*0.0675} 0.084" rpy="0 0 0"/>
-			<axis xyz="0 1 0"/>
+			<axis xyz="0 ${reflect*1} 0"/>
 			<limit lower="-3.14159265" upper="3.14159265" effort="6.0" velocity="6.597344565"/>
 		</joint>
@@ -40,5 +40,5 @@
 		<child link="LUpperArm"/>
 		<origin xyz="0.002 0.03 -0.03" rpy="${PI_2/2} 0 0"/>
-		<axis xyz="1 0 0"/>
+		<axis xyz="-1 0 0"/>
 		<limit lower="-2.35619449" upper="1.30899694" effort="6.0" velocity="6.597344565"/>
 	</joint>
@@ -47,5 +47,5 @@
 		<child link="RUpperArm"/>
 		<origin xyz="0.002 -0.03 -0.03" rpy="-${PI_2/2} 0 0"/>
-		<axis xyz="1 0 0"/>
+		<axis xyz="-1 0 0"/>
 		<limit lower="-1.30899694" upper="2.35619449" effort="6.0" velocity="6.597344565"/>
 	</joint>
@@ -54,5 +54,5 @@
 		<child link="LLowerArm"/>
 		<origin xyz="0.03 -0.0015 -0.085" rpy="0 -${PI_2/2} 0"/>
-		<axis xyz="0 1 0"/>
+		<axis xyz="0 -1 0"/>
 		<limit lower="-1.22173048" upper="1.65806279" effort="6.0" velocity="6.597344565"/>
 	</joint>

File: hros5_description/urdf/modules/head.xacro (robot description, xacro)
@@ -6,5 +6,5 @@
 		<origin xyz="0.0035 0 0.1115" rpy="0 0 0"/>
 		<axis xyz="0 0 1"/>
-		<limit lower="-1.22173048" upper="1.22173048" effort="2.5" velocity="5.759586525"/>
+		<limit lower="-2.6179939" upper="2.6179939" effort="2.5" velocity="5.759586525"/>
 	</joint>
 	<link name="LowerHead">
@@ -20,5 +20,5 @@
 		<child link="UpperHeadBase"/>
 		<origin xyz="-0.01 0 0.049" rpy="0 0 0"/>
-		<axis xyz="0 1 0"/>
+		<axis xyz="0 -1 0"/>
 		<limit upper="0.4" lower="-0.25" effort="2.5" velocity="5.759586525"/>
 	</joint>
@@ -36,5 +36,5 @@
 		<origin xyz="-0.00225 0 0.046" rpy="0 0 0"/>
 		<axis xyz="0 1 0"/>
-		<mimic joint="HeadPitch" multiplier="-1.0"/>
+		<mimic joint="HeadPitch" multiplier="1.0"/>
 	</joint>
 	<link name="UpperHeadMotor">
@@ -51,5 +51,5 @@
 		<origin xyz="-0.0525 0 0.021" rpy="0 0 0"/>
 		<axis xyz="0 1 0"/>
-		<mimic joint="HeadPitch" multiplier="0.65"/>
+		<mimic joint="HeadPitch" multiplier="-0.65"/>
 	</joint>
 	<link name="UpperHeadBack">
@@ -61,4 +61,32 @@
 		</inertial>
 	</link>
+<!-- Camera properties -->
+<xacro:property name="pi" value="3.1415926535897931" />
+<!-- openni2 / primesense on top of servo -->
+<joint name="camera_rgb_joint" type="fixed">
+	<parent link="UpperHeadBase" />
+	<child link="camera_rgb_optical_frame" />
+	<origin xyz="0.0 0.0 0.08" rpy="${pi/2} ${pi} ${pi/2}" />
+</joint>
+<link name="camera_rgb_optical_frame" />
+<joint name="camera_depth_joint" type="fixed">
+	<parent link="UpperHeadBase" />
+	<child link="camera_depth_optical_frame" />
+	<origin xyz="0.0 0.0 0.08" rpy="${pi/2} ${pi} ${pi/2}" />
+</joint>
+<link name="camera_depth_optical_frame" />
+<joint name="camera_depth_frame" type="fixed">
+	<parent link="UpperHeadBase" />
+	<child link="camera_depth_frame_link" />
+	<origin xyz="0.0 0.0 0.08" />
+</joint>
+<link name="camera_depth_frame_link" />
+<!-- intel r200 on front of servo -->
+<joint name="r200_frame" type="fixed">
+	<parent link="UpperHeadBase" />
+	<child link="realsense_frame" />
+	<origin xyz="0.05 -0.05 0.05" rpy="${pi/2} ${pi} ${pi/2}" />
+</joint>
+<link name="realsense_frame" />
 <!-- ROS REP LINKS -->
 	<joint name="gaze_joint" type="fixed">

File: hros5_description/urdf/modules/legs.xacro (robot description, xacro)
@@ -36,5 +36,5 @@
 			<child link="${side}Thigh"/>
 			<origin xyz="0.0705 0 0" rpy="0 0 0"/>
-			<axis xyz="0 1 0"/>
+			<axis xyz="0 ${reflect*-1} 0"/>
 			<limit lower="-1.57079633" upper="1.57079633" effort="8.4" velocity="4.712388975"/>
 		</joint>
@@ -51,5 +51,5 @@
 			<child link="${side}Tibia"/>
 			<origin xyz="0.0017 0 -0.127" rpy="0 0 0"/>
-			<axis xyz="0 1 0"/>
+			<axis xyz="0 ${reflect*-1} 0"/>
 			<limit lower="-2.7925268" upper="2.7925268" effort="8.4" velocity="4.712388975"/>
 		</joint>
@@ -66,5 +66,5 @@
 			<child link="${side}Ankle"/>
 			<origin xyz="-0.002 0 -0.125" rpy="0 0 0"/>
-			<axis xyz="0 1 0"/>
+			<axis xyz="0 ${reflect*1} 0"/>
 			<limit lower="-1.57079633" upper="1.57079633" effort="8.4" velocity="4.712388975"/>
 		</joint>
@@ -81,5 +81,5 @@
 			<child link="${side}Foot"/>
 			<origin xyz="-0.07 0 0" rpy="0 0 0"/>
-			<axis xyz="1 0 0"/>
+			<axis xyz="-1 0 0"/>
 			<limit lower="-0.785398163" upper="0.785398163" effort="8.4" velocity="4.712388975"/>
 		</joint>

File: hros5_description/urdf/modules/torso.xacro (robot description, xacro)
@@ -1,9 +1,9 @@
 <?xml version="1.0"?>
 <robot xmlns:xacro="http://www.ros.org/wiki/xacro">
-	<!-- DUMMY ROOT LINK -->
 	<link name="base_link"/>
-	<joint name="fixed-base" type="fixed">
+	<joint name="base_joint" type="fixed">
 		<parent link="base_link"/>
 		<child link="torso"/>
+		<origin xyz="0 0 0.024" rpy="0 0 0"/>
 	</joint>
 	<!-- TORSO -->
@@ -16,3 +16,32 @@
 		</inertial>
 	</link>
+<!-- IMU properties -->
+<joint name="imu_joint" type="floating">
+    <parent link="base_link"/>
+    <child link="torso"/>
+    <origin xyz="0.0 0.0 0.033" rpy="0.0 0.0 0.0"/>
+</joint>
+<!--
+<link name="imu_link">
+    <inertial>
+        <origin xyz="0.0 0.0 0.0" rpy="0.0 0.0 0.0" />
+        <mass value="0.00001"/>
+        <inertia
+            ixx="1.0" ixy="0.0"  ixz="0.0"
+            iyy="1.0" iyz="0.0"
+            izz="1.0" />
+    </inertial>
+</link>
+-->
+	<gazebo>
+        <plugin filename="libhector_gazebo_ros_imu.so" name="gazebo_ros_imu">
+          <bodyName>torso</bodyName>
+          <updateRate>50</updateRate>
+          <serviceName>/hros5/imu_service</serviceName>
+          <topicName>/hros5/imu</topicName>
+          <gaussianNoise>0</gaussianNoise>
+          <xyzOffset>0 0 0</xyzOffset>
+          <rpyOffset>0 0 -0.703220730592</rpyOffset>
+        </plugin>
+      </gazebo>
 </robot>
